Commit message: Internal changes from Intrinsic
GitOrigin-RevId: 173f9ae95684715176376dfd4cff92529fc80bfe

File: intrinsic_control/intrinsic/models/robot_definitions/fanuc/crx_10ia/crx_10ia.xacro (robot description, xacro)
@@ -13,5 +13,5 @@
 <sdf version='1.9' xmlns:xacro='http://www.ros.org/wiki/xacro'>
 <xacro:include filename="$(cwd)/third_party/fanuc/crx_10ia/crx_10ia_base.xacro"/>
-<xacro:include filename="$(cwd)/intrinsic_control/intrinsic/models/robot_definitions/fanuc/simulation_plugins.xacro"/>
+<xacro:include filename="$(cwd)/intrinsic_control/intrinsic/models/robot_definitions/fanuc/timeslicer_plugins.xacro"/>
 <!-- Expands to an Fanuc crx_10ia robot that can be customized with various
   options like starting pose.
@@ -24,4 +24,5 @@
       </model_options>
     </xacro:crx_10ia_sdf>
+  joint_*_initial: Initial joint positions of the generated robot (in radians).
 -->
 <xacro:macro name='crx_10ia_sdf' params='name
@@ -29,5 +30,5 @@
   <xacro:crx_10ia_base_sdf name="${name}">
     <model_options>
-      <xacro:simulation_plugins/>
+      <xacro:timeslicer_plugins />
       <!-- Append passed in model options. -->
       <xacro:insert_block name="model_options"/>

File: intrinsic_control/intrinsic/models/robot_definitions/fanuc/crx_10ia_l/crx_10ia_l.xacro (robot description, xacro)
@@ -13,5 +13,5 @@
 <sdf version='1.9' xmlns:xacro='http://www.ros.org/wiki/xacro'>
 <xacro:include filename="$(cwd)/third_party/fanuc/crx_10ia_l/crx_10ia_l_base.xacro"/>
-<xacro:include filename="$(cwd)/intrinsic_control/intrinsic/models/robot_definitions/fanuc/simulation_plugins.xacro"/>
+<xacro:include filename="$(cwd)/intrinsic_control/intrinsic/models/robot_definitions/fanuc/timeslicer_plugins.xacro"/>
 <!-- Expands to an Fanuc crx_10ia_l robot that can be customized with various
   options like starting pose.
@@ -24,4 +24,5 @@
       </model_options>
     </xacro:crx_10ia_l_sdf>
+  joint_*_initial: Initial joint positions of the generated robot (in radians).
 -->
 <xacro:macro name='crx_10ia_l_sdf' params='name
@@ -29,5 +30,5 @@
   <xacro:crx_10ia_l_base_sdf name="${name}">
     <model_options>
-      <xacro:simulation_plugins/>
+      <xacro:timeslicer_plugins />
       <!-- Append passed in model options. -->
       <xacro:insert_block name="model_options"/>

File: intrinsic_control/intrinsic/models/robot_definitions/fanuc/crx_20ia_l/crx_20ia_l.xacro (robot description, xacro)
@@ -13,5 +13,5 @@
 <sdf version='1.9' xmlns:xacro='http://www.ros.org/wiki/xacro'>
 <xacro:include filename="$(cwd)/third_party/fanuc/crx_20ia_l/crx_20ia_l_base.xacro"/>
-<xacro:include filename="$(cwd)/intrinsic_control/intrinsic/models/robot_definitions/fanuc/simulation_plugins.xacro"/>
+<xacro:include filename="$(cwd)/intrinsic_control/intrinsic/models/robot_definitions/fanuc/timeslicer_plugins.xacro"/>
 <!-- Expands to an Fanuc crx_20ia_l robot that can be customized with various
   options like starting pose.
@@ -24,4 +24,5 @@
       </model_options>
     </xacro:crx_20ia_l_sdf>
+  joint_*_initial: Initial joint positions of the generated robot (in radians).
 -->
 <xacro:macro name='crx_20ia_l_sdf' params='name
@@ -29,5 +30,5 @@
   <xacro:crx_20ia_l_base_sdf name="${name}">
     <model_options>
-      <xacro:simulation_plugins/>
+      <xacro:timeslicer_plugins />
       <!-- Append passed in model options. -->
       <xacro:insert_block name="model_options"/>

File: intrinsic_control/intrinsic/models/robot_definitions/fanuc/crx_30ia/crx_30ia.xacro (robot description, xacro)
@@ -13,5 +13,5 @@
 <sdf version='1.9' xmlns:xacro='http://www.ros.org/wiki/xacro'>
 <xacro:include filename="$(cwd)/third_party/fanuc/crx_30ia/crx_30ia_base.xacro"/>
-<xacro:include filename="$(cwd)/intrinsic_control/intrinsic/models/robot_definitions/fanuc/simulation_plugins.xacro"/>
+<xacro:include filename="$(cwd)/intrinsic_control/intrinsic/models/robot_definitions/fanuc/timeslicer_plugins.xacro"/>
 <!-- Expands to an Fanuc crx_30ia robot that can be customized with various
   options like starting pose.
@@ -30,5 +30,5 @@
   <xacro:crx_30ia_base_sdf name="${name}">
     <model_options>
-      <xacro:simulation_plugins/>
+      <xacro:timeslicer_plugins />
       <!-- Append passed in model options. -->
       <xacro:insert_block name="model_options"/>

File: intrinsic_control/intrinsic/models/robot_definitions/fanuc/lr_10ia_10/lr_10ia_10.xacro (robot description, xacro)
@@ -13,5 +13,5 @@
 <sdf version='1.9' xmlns:xacro='http://www.ros.org/wiki/xacro'>
 <xacro:include filename="$(cwd)/third_party/fanuc/lr_10ia_10/lr_10ia_10_base.xacro"/>
-<xacro:include filename="$(cwd)/intrinsic_control/intrinsic/models/robot_definitions/fanuc/simulation_plugins.xacro"/>
+<xacro:include filename="$(cwd)/intrinsic_control/intrinsic/models/robot_definitions/fanuc/timeslicer_plugins.xacro"/>
 <!-- Expands to an Fanuc lr_10ia_10 robot that can be customized with various
   options like starting pose.
@@ -24,4 +24,5 @@
       </model_options>
     </xacro:lr_10ia_10_sdf>
+  joint_*_initial: Initial joint positions of the generated robot (in radians).
 -->
 <xacro:macro name='lr_10ia_10_sdf' params='name
@@ -29,5 +30,5 @@
   <xacro:lr_10ia_10_base_sdf name="${name}">
     <model_options>
-      <xacro:simulation_plugins/>
+      <xacro:timeslicer_plugins />
       <!-- Append passed in model options. -->
       <xacro:insert_block name="model_options"/>

File: intrinsic_control/intrinsic/models/robot_definitions/fanuc/lr_mate_200id/lr_mate_200id.xacro (robot description, xacro)
@@ -13,5 +13,5 @@
 <sdf version='1.9' xmlns:xacro='http://www.ros.org/wiki/xacro'>
 <xacro:include filename="$(cwd)/third_party/fanuc/lr_mate_200id/lr_mate_200id_base.xacro"/>
-<xacro:include filename="$(cwd)/intrinsic_control/intrinsic/models/robot_definitions/fanuc/simulation_plugins.xacro"/>
+<xacro:include filename="$(cwd)/intrinsic_control/intrinsic/models/robot_definitions/fanuc/timeslicer_plugins.xacro"/>
 <!-- Expands to an Fanuc lr_mate_200id robot that can be customized with various
   options like starting pose.
@@ -24,4 +24,5 @@
       </model_options>
     </xacro:lr_mate_200id_sdf>
+  joint_*_initial: Initial joint positions of the generated robot (in radians).
 -->
 <xacro:macro name='lr_mate_200id_sdf' params='name
@@ -29,5 +30,5 @@
   <xacro:lr_mate_200id_base_sdf name="${name}">
     <model_options>
-      <xacro:simulation_plugins/>
+      <xacro:timeslicer_plugins />
       <!-- Append passed in model options. -->
       <xacro:insert_block name="model_options"/>

File: intrinsic_control/intrinsic/models/robot_definitions/fanuc/lr_mate_200id_4s/lr_mate_200id_4s.xacro (robot description, xacro)
@@ -13,5 +13,5 @@
 <sdf version='1.9' xmlns:xacro='http://www.ros.org/wiki/xacro'>
 <xacro:include filename="$(cwd)/third_party/fanuc/lr_mate_200id_4s/lr_mate_200id_4s_base.xacro"/>
-<xacro:include filename="$(cwd)/intrinsic_control/intrinsic/models/robot_definitions/fanuc/simulation_plugins.xacro"/>
+<xacro:include filename="$(cwd)/intrinsic_control/intrinsic/models/robot_definitions/fanuc/timeslicer_plugins.xacro"/>
 <!-- Expands to an Fanuc lr_mate_200id_4s robot that can be customized with various
   options like starting pose.
@@ -24,4 +24,5 @@
       </model_options>
     </xacro:lr_mate_200id_4s_sdf>
+  joint_*_initial: Initial joint positions of the generated robot (in radians).
 -->
 <xacro:macro name='lr_mate_200id_4s_sdf' params='name
@@ -29,5 +30,5 @@
   <xacro:lr_mate_200id_4s_base_sdf name="${name}">
     <model_options>
-      <xacro:simulation_plugins/>
+      <xacro:timeslicer_plugins />
       <!-- Append passed in model options. -->
       <xacro:insert_block name="model_options"/>

File: intrinsic_control/intrinsic/models/robot_definitions/fanuc/lr_mate_200id_7l/lr_mate_200id_7l.xacro (robot description, xacro)
@@ -13,5 +13,5 @@
 <sdf version='1.9' xmlns:xacro='http://www.ros.org/wiki/xacro'>
 <xacro:include filename="$(cwd)/third_party/fanuc/lr_mate_200id_7l/lr_mate_200id_7l_base.xacro"/>
-<xacro:include filename="$(cwd)/intrinsic_control/intrinsic/models/robot_definitions/fanuc/simulation_plugins.xacro"/>
+<xacro:include filename="$(cwd)/intrinsic_control/intrinsic/models/robot_definitions/fanuc/timeslicer_plugins.xacro"/>
 <!-- Expands to an Fanuc lr_mate_200id_7l robot that can be customized with various
   options like starting pose.
@@ -24,4 +24,5 @@
       </model_options>
     </xacro:lr_mate_200id_7l_sdf>
+  joint_*_initial: Initial joint positions of the generated robot (in radians).
 -->
 <xacro:macro name='lr_mate_200id_7l_sdf' params='name
@@ -29,5 +30,5 @@
   <xacro:lr_mate_200id_7l_base_sdf name="${name}">
     <model_options>
-      <xacro:simulation_plugins/>
+      <xacro:timeslicer_plugins />
       <!-- Append passed in model options. -->
       <xacro:insert_block name="model_options"/>

File: intrinsic_control/intrinsic/models/robot_definitions/fanuc/m_10id_12/m_10id_12.xacro (robot description, xacro)
@@ -13,5 +13,5 @@
 <sdf version='1.9' xmlns:xacro='http://www.ros.org/wiki/xacro'>
 <xacro:include filename="$(cwd)/third_party/fanuc/m_10id_12/m_10id_12_base.xacro"/>
-<xacro:include filename="$(cwd)/intrinsic_control/intrinsic/models/robot_definitions/fanuc/simulation_plugins.xacro"/>
+<xacro:include filename="$(cwd)/intrinsic_control/intrinsic/models/robot_definitions/fanuc/timeslicer_plugins.xacro"/>
 <!-- Expands to an Fanuc m_10id_12 robot that can be customized with various
   options like starting pose.
@@ -24,4 +24,5 @@
       </model_options>
     </xacro:m_10id_12_sdf>
+  joint_*_initial: Initial joint positions of the generated robot (in radians).
 -->
 <xacro:macro name='m_10id_12_sdf' params='name
@@ -29,5 +30,5 @@
   <xacro:m_10id_12_base_sdf name="${name}">
     <model_options>
-      <xacro:simulation_plugins/>
+      <xacro:timeslicer_plugins />
       <!-- Append passed in model options. -->
       <xacro:insert_block name="model_options"/>

File: intrinsic_control/intrinsic/models/robot_definitions/fanuc/m_20id/m_20id.xacro (robot description, xacro)
@@ -13,5 +13,5 @@
 <sdf version='1.9' xmlns:xacro='http://www.ros.org/wiki/xacro'>
 <xacro:include filename="$(cwd)/third_party/fanuc/m_20id/m_20id_base.xacro"/>
-<xacro:include filename="$(cwd)/intrinsic_control/intrinsic/models/robot_definitions/fanuc/simulation_plugins.xacro"/>
+<xacro:include filename="$(cwd)/intrinsic_control/intrinsic/models/robot_definitions/fanuc/timeslicer_plugins.xacro"/>
 <!-- Expands to an Fanuc m_20id robot that can be customized with various
   options like starting pose.
@@ -24,4 +24,5 @@
       </model_options>
     </xacro:m_20id_sdf>
+  joint_*_initial: Initial joint positions of the generated robot (in radians).
 -->
 <xacro:macro name='m_20id_sdf' params='name
@@ -29,5 +30,5 @@
   <xacro:m_20id_base_sdf name="${name}">
     <model_options>
-      <xacro:simulation_plugins/>
+      <xacro:timeslicer_plugins />
       <!-- Append passed in model options. -->
       <xacro:insert_block name="model_options"/>

File: intrinsic_control/intrinsic/models/robot_definitions/fanuc/m_710id_50m/m_710id_50m.xacro (robot description, xacro)
@@ -13,5 +13,5 @@
 <sdf version='1.9' xmlns:xacro='http://www.ros.org/wiki/xacro'>
 <xacro:include filename="$(cwd)/third_party/fanuc/m_710id_50m/m_710id_50m_base.xacro"/>
-<xacro:include filename="$(cwd)/intrinsic_control/intrinsic/models/robot_definitions/fanuc/simulation_plugins.xacro"/>
+<xacro:include filename="$(cwd)/intrinsic_control/intrinsic/models/robot_definitions/fanuc/timeslicer_plugins.xacro"/>
 <!-- Expands to an Fanuc m_710id_50m robot that can be customized with various
   options like starting pose.
@@ -24,4 +24,5 @@
       </model_options>
     </xacro:m_710id_50m_sdf>
+  joint_*_initial: Initial joint positions of the generated robot (in radians).
 -->
 <xacro:macro name='m_710id_50m_sdf' params='name
@@ -29,5 +30,5 @@
   <xacro:m_710id_50m_base_sdf name="${name}">
     <model_options>
-      <xacro:simulation_plugins/>
+      <xacro:timeslicer_plugins />
       <!-- Append passed in model options. -->
       <xacro:insert_block name="model_options"/>

File: intrinsic_control/intrinsic/models/robot_definitions/fanuc/r_2000ic_210l/r_2000ic_210l.xacro (robot description, xacro)
@@ -13,5 +13,5 @@
 <sdf version='1.9' xmlns:xacro='http://www.ros.org/wiki/xacro'>
 <xacro:include filename="$(cwd)/third_party/fanuc/r_2000ic_210l/r_2000ic_210l_base.xacro"/>
-<xacro:include filename="$(cwd)/intrinsic_control/intrinsic/models/robot_definitions/fanuc/simulation_plugins.xacro"/>
+<xacro:include filename="$(cwd)/intrinsic_control/intrinsic/models/robot_definitions/fanuc/timeslicer_plugins.xacro"/>
 <!-- Expands to an Fanuc r_2000ic_210l robot that can be customized with various
   options like starting pose.
@@ -24,4 +24,5 @@
       </model_options>
     </xacro:r_2000ic_210l_sdf>
+  joint_*_initial: Initial joint positions of the generated robot (in radians).
 -->
 <xacro:macro name='r_2000ic_210l_sdf' params='name
@@ -29,5 +30,5 @@
   <xacro:r_2000ic_210l_base_sdf name="${name}">
     <model_options>
-      <xacro:simulation_plugins/>
+      <xacro:timeslicer_plugins />
       <!-- Append passed in model options. -->
       <xacro:insert_block name="model_options"/>

File: intrinsic_control/intrinsic/models/robot_definitions/fanuc/timeslicer_plugins.xacro (robot description, xacro)
@@ -12,5 +12,7 @@
 -->
 <sdf version='1.6' xmlns:xacro='http://www.ros.org/wiki/xacro'>
-  <xacro:macro name="simulation_plugins">
+  <xacro:macro name="timeslicer_plugins">
+    <plugin filename="static://intrinsic::simulation::TimeslicerWorld" name="TimeslicerPlugin">
+    </plugin>
     <!-- HAL Digital IO Block simulation -->
     <plugin filename="static://intrinsic::simulation::DigitalInputOutput" name="DigitalInputOutput">
